File: pcb/UsbDmx.sch (EAGLE design)
At the start: 22 parts, among them IC4 SN75176ASOIC, J2 POWER_JACKPTH, X1 USBPTH

Commit message: Replaced crystal with smaller 3025 version, placed and routed all passives.
TODO: finish routing processor ground, final check, assemble BOM.
Parts:
- removed Q2: (no value), blinkyboard:GLOWBOARD_ABMM2
- added Q1: (no value), blinkyboard:CRYSTAL
Connections:
- removed net D4: R3.2, R8.2
- new net D10: R3.2, U$1.(PCINT6/OC1B/OC4B/ADC13)PB6
- new net D9: R8.2, U$1.(PCINT5/OC1A/#OC4B/ADC12)PB5
- net N$2: now also Q1.2; no longer Q2.2
- net N$5: now also Q1.1; no longer Q2.1
Changed lines of the file:
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@@
 <part name="C1" library="SparkFun" deviceset="CAP" device="0805" value="16pf"/>
 <part name="C2" library="SparkFun" deviceset="CAP" device="0805" value="16pf"/>
-<part name="Q2" library="blinkyboard" deviceset="GLOWBOARD_ABMM2" device=""/>
 <part name="GND5" library="supply1" deviceset="GND" device=""/>
 <part name="R4" library="SparkFun" deviceset="RESISTOR" device="" value="10K"/>
@@
 <part name="GND4" library="supply1" deviceset="GND" device=""/>
 <part name="P+2" library="supply1" deviceset="VCC" device=""/>
+<part name="Q1" library="blinkyboard" deviceset="CRYSTAL" device=""/>
 </parts>
 <sheets>
@@
 <instance part="C1" gate="G$1" x="-17.78" y="45.72" rot="R90"/>
 <instance part="C2" gate="G$1" x="-17.78" y="35.56" rot="R90"/>
-<instance part="Q2" gate="G$1" x="-10.16" y="40.64" rot="R90"/>
 <instance part="GND5" gate="1" x="-25.4" y="30.48"/>
 <instance part="R4" gate="G$1" x="0" y="60.96" rot="R90"/>
@@
 <instance part="GND4" gate="1" x="-12.7" y="-25.4"/>
 <instance part="P+2" gate="VCC" x="-12.7" y="-7.62"/>
+<instance part="Q1" gate="G$1" x="-10.16" y="40.64" rot="R90"/>
 </instances>
 <busses>
@@
 <wire x1="73.66" y1="0" x2="76.2" y2="0" width="0.1524" layer="91"/>
 <label x="76.2" y="0" size="1.778" layer="95" xref="yes"/>
-</segment>
-</net>
-<net name="D4" class="0">
-<segment>
-<wire x1="157.48" y1="15.24" x2="157.48" y2="20.32" width="0.1524" layer="91"/>
-<label x="157.48" y="20.32" size="1.778" layer="95" rot="R90" xref="yes"/>
-<pinref part="R8" gate="G$1" pin="2"/>
-</segment>
-<segment>
-<wire x1="167.64" y1="15.24" x2="167.64" y2="20.32" width="0.1524" layer="91"/>
-<label x="167.64" y="20.32" size="1.778" layer="95" rot="R90" xref="yes"/>
-<pinref part="R3" gate="G$1" pin="2"/>
 </segment>
 </net>
@@
 <wire x1="-15.24" y1="45.72" x2="-10.16" y2="45.72" width="0.1524" layer="91"/>
 <pinref part="C1" gate="G$1" pin="2"/>
-<pinref part="Q2" gate="G$1" pin="2"/>
-<junction x="-10.16" y="45.72"/>
 <pinref part="U$1" gate="G$1" pin="XTAL2"/>
 <wire x1="12.7" y1="45.72" x2="-10.16" y2="45.72" width="0.1524" layer="91"/>
+<pinref part="Q1" gate="G$1" pin="2"/>
+<wire x1="-10.16" y1="43.18" x2="-10.16" y2="45.72" width="0.1524" layer="91"/>
+<junction x="-10.16" y="45.72"/>
 </segment>
 </net>
@@
 <segment>
 <pinref part="C2" gate="G$1" pin="2"/>
-<pinref part="Q2" gate="G$1" pin="1"/>
 <wire x1="-15.24" y1="35.56" x2="-10.16" y2="35.56" width="0.1524" layer="91"/>
 <wire x1="-10.16" y1="35.56" x2="-5.08" y2="35.56" width="0.1524" layer="91"/>
 <wire x1="-5.08" y1="35.56" x2="-5.08" y2="40.64" width="0.1524" layer="91"/>
-<junction x="-10.16" y="35.56"/>
 <pinref part="U$1" gate="G$1" pin="XTAL1"/>
 <wire x1="-5.08" y1="40.64" x2="12.7" y2="40.64" width="0.1524" layer="91"/>
+<pinref part="Q1" gate="G$1" pin="1"/>
+<wire x1="-10.16" y1="38.1" x2="-10.16" y2="35.56" width="0.1524" layer="91"/>
+<junction x="-10.16" y="35.56"/>
 </segment>
 </net>
@@
 </segment>
 </net>
+<net name="D9" class="0">
+<segment>
+<pinref part="U$1" gate="G$1" pin="(PCINT5/OC1A/#OC4B/ADC12)PB5"/>
+<wire x1="73.66" y1="53.34" x2="76.2" y2="53.34" width="0.1524" layer="91"/>
+<label x="76.2" y="53.34" size="1.778" layer="95" xref="yes"/>
+</segment>
+<segment>
+<wire x1="157.48" y1="15.24" x2="157.48" y2="20.32" width="0.1524" layer="91"/>
+<label x="157.48" y="20.32" size="1.778" layer="95" rot="R90" xref="yes"/>
+<pinref part="R8" gate="G$1" pin="2"/>
+</segment>
+</net>
+<net name="D10" class="0">
+<segment>
+<pinref part="U$1" gate="G$1" pin="(PCINT6/OC1B/OC4B/ADC13)PB6"/>
+<wire x1="73.66" y1="55.88" x2="76.2" y2="55.88" width="0.1524" layer="91"/>
+<label x="76.2" y="55.88" size="1.778" layer="95" xref="yes"/>
+</segment>
+<segment>
+<wire x1="167.64" y1="15.24" x2="167.64" y2="20.32" width="0.1524" layer="91"/>
+<label x="167.64" y="20.32" size="1.778" layer="95" rot="R90" xref="yes"/>
+<pinref part="R3" gate="G$1" pin="2"/>
+</segment>
+</net>

Commit message: Fixed processor thermal vias (no more DRC errors), finished ground routing, added missing UCAP
Parts:
- added C4: 1uF, SparkFun:CAP0805
- added JP1: (no value), SparkFun:M02PTH
- DEBUG: value (none) -> RED
- DEBUG1: value (none) -> GREEN
- J1: value (none) -> RS485
- Q1: value (none) -> 16MHz 10ppm
- U$1: device blinkyboard:ARDUINO_LEONARDO-REV3B_SMARTPRJ_ATMEGA32U4-XUMU -> blinkiverse:ARDUINO_LEONARDO-REV3B_SMARTPRJ_ATMEGA32U4-XUMU
Connections:
- removed net D2: U$1.(SDA/INT1)PD1
- new net A2: JP1.2, U$1.(ADC5/TMS)PF5
- new net A3: JP1.1, U$1.(ADC4/TCK)PF4
- new net N$9: C4.2, U$1.UCAP
- net GND: now also C4.1
Other:
- note added: "EXTRA"
- moved on the sheet: R5, R6, U$1
Changed lines of the file:
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@@
 <part name="R2" library="SparkFun" deviceset="RESISTOR" device="" value="10k"/>
 <part name="R8" library="SparkFun" deviceset="RESISTOR" device="" value="1K"/>
-<part name="DEBUG" library="SparkFun" deviceset="LED" device="0805"/>
+<part name="DEBUG" library="SparkFun" deviceset="LED" device="0805" value="RED"/>
 <part name="GND12" library="supply1" deviceset="GND" device=""/>
 <part name="P+14" library="supply1" deviceset="VCC" device=""/>
 <part name="C7" library="SparkFun" deviceset="CAP" device="0805" value="100nF"/>
 <part name="GND8" library="SparkFun" deviceset="GND" device=""/>
-<part name="J1" library="con-amp" deviceset="520426-4" device=""/>
+<part name="J1" library="con-amp" deviceset="520426-4" device="" value="RS485"/>
 <part name="U$2" library="sonos_library" deviceset="2X3HEADER" device=""/>
 <part name="P+5" library="supply1" deviceset="VCC" device=""/>
 <part name="GND10" library="supply1" deviceset="GND" device=""/>
-<part name="U$1" library="blinkyboard" deviceset="ARDUINO_LEONARDO-REV3B_SMARTPRJ_ATMEGA32U4-XU" device="MU"/>
+<part name="U$1" library="blinkiverse" deviceset="ARDUINO_LEONARDO-REV3B_SMARTPRJ_ATMEGA32U4-XU" device="MU"/>
 <part name="P+1" library="supply1" deviceset="VCC" device=""/>
 <part name="GND1" library="supply1" deviceset="GND" device=""/>
@@
 <part name="R6" library="SparkFun" deviceset="RESISTOR" device="" value="22"/>
 <part name="R3" library="SparkFun" deviceset="RESISTOR" device="" value="1K"/>
-<part name="DEBUG1" library="SparkFun" deviceset="LED" device="0805"/>
+<part name="DEBUG1" library="SparkFun" deviceset="LED" device="0805" value="GREEN"/>
 <part name="GND3" library="supply1" deviceset="GND" device=""/>
 <part name="C3" library="SparkFun" deviceset="CAP" device="0805" value=".1uF"/>
@@
 <part name="GND4" library="supply1" deviceset="GND" device=""/>
 <part name="P+2" library="supply1" deviceset="VCC" device=""/>
-<part name="Q1" library="blinkyboard" deviceset="CRYSTAL" device=""/>
+<part name="Q1" library="blinkyboard" deviceset="CRYSTAL" device="" value="16MHz 10ppm"/>
+<part name="JP1" library="SparkFun" deviceset="M02" device="PTH"/>
+<part name="C4" library="SparkFun" deviceset="CAP" device="0805" value="1uF"/>
+<part name="GND6" library="supply1" deviceset="GND" device=""/>
 </parts>
 <sheets>
@@
 <wire x1="101.6" y1="35.56" x2="101.6" y2="2.54" width="0.4064" layer="94"/>
 <wire x1="101.6" y1="2.54" x2="147.32" y2="2.54" width="0.4064" layer="94"/>
-<wire x1="147.32" y1="2.54" x2="147.32" y2="35.56" width="0.4064" layer="94"/>
 <wire x1="180.34" y1="35.56" x2="149.86" y2="35.56" width="0.4064" layer="94"/>
 <wire x1="149.86" y1="35.56" x2="149.86" y2="-17.78" width="0.4064" layer="94"/>
@@
 <text x="152.4" y="30.48" size="2.54" layer="94">INDICATOR</text>
 <wire x1="-30.48" y1="78.74" x2="-30.48" y2="-33.02" width="0.4064" layer="94"/>
+<text x="104.14" y="-5.08" size="2.54" layer="94">EXTRA</text>
+<wire x1="147.32" y1="0" x2="101.6" y2="0" width="0.4064" layer="94"/>
+<wire x1="101.6" y1="0" x2="101.6" y2="-20.32" width="0.4064" layer="94"/>
+<wire x1="147.32" y1="2.54" x2="147.32" y2="35.56" width="0.4064" layer="94"/>
+<wire x1="147.32" y1="-20.32" x2="147.32" y2="0" width="0.4064" layer="94"/>
+<wire x1="101.6" y1="-20.32" x2="147.32" y2="-20.32" width="0.4064" layer="94"/>
 </plain>
 <instances>
@@
 <instance part="GND5" gate="1" x="-25.4" y="30.48"/>
 <instance part="R4" gate="G$1" x="0" y="60.96" rot="R90"/>
-<instance part="X1" gate="G$1" x="-15.24" y="15.24" rot="R180"/>
+<instance part="X1" gate="G$1" x="-20.32" y="15.24" rot="R180"/>
 <instance part="J2" gate="G$1" x="180.34" y="66.04" rot="R180"/>
-<instance part="R5" gate="G$1" x="-5.08" y="7.62"/>
-<instance part="R6" gate="G$1" x="-5.08" y="10.16"/>
+<instance part="R5" gate="G$1" x="-10.16" y="7.62"/>
+<instance part="R6" gate="G$1" x="-10.16" y="10.16"/>
 <instance part="R3" gate="G$1" x="167.64" y="10.16" rot="R90"/>
 <instance part="DEBUG1" gate="G$1" x="167.64" y="0"/>
@@
 <instance part="P+2" gate="VCC" x="-12.7" y="-7.62"/>
 <instance part="Q1" gate="G$1" x="-10.16" y="40.64" rot="R90"/>
+<instance part="JP1" gate="G$1" x="127" y="-10.16" rot="R180"/>
+<instance part="C4" gate="G$1" x="0" y="30.48" smashed="yes" rot="R180">
+<attribute name="NAME" x="-4.064" y="30.099" size="1.778" layer="95" rot="R180"/>
+<attribute name="VALUE" x="-1.524" y="32.639" size="1.778" layer="96" rot="R180"/>
+</instance>
+<instance part="GND6" gate="1" x="0" y="20.32"/>
 </instances>
 <busses>
@@
 <wire x1="177.8" y1="63.5" x2="162.56" y2="63.5" width="0.1524" layer="91"/>
 <junction x="162.56" y="63.5"/>
+<junction x="177.8" y="63.5"/>
 </segment>
 <segment>
@@
 <junction x="10.16" y="22.86"/>
 <pinref part="X1" gate="G$1" pin="GND"/>
-<wire x1="-12.7" y1="15.24" x2="5.08" y2="15.24" width="0.1524" layer="91"/>
-<wire x1="5.08" y1="15.24" x2="5.08" y2="5.08" width="0.1524" layer="91"/>
-<wire x1="5.08" y1="5.08" x2="10.16" y2="5.08" width="0.1524" layer="91"/>
+<wire x1="-17.78" y1="15.24" x2="0" y2="15.24" width="0.1524" layer="91"/>
+<wire x1="0" y1="15.24" x2="0" y2="5.08" width="0.1524" layer="91"/>
+<wire x1="0" y1="5.08" x2="10.16" y2="5.08" width="0.1524" layer="91"/>
 </segment>
 <segment>
@@
 <junction x="-12.7" y="-20.32"/>
 </segment>
+<segment>
+<pinref part="C4" gate="G$1" pin="1"/>
+<pinref part="GND6" gate="1" pin="GND"/>
+<wire x1="0" y1="25.4" x2="0" y2="22.86" width="0.1524" layer="91"/>
+</segment>
 </net>
 <net name="RX" class="0">
@@
 <wire x1="73.66" y1="7.62" x2="76.2" y2="7.62" width="0.1524" layer="91"/>
 <label x="76.2" y="7.62" size="1.778" layer="95" xref="yes"/>
-</segment>
-</net>
-<net name="D2" class="0">
-<segment>
-<pinref part="U$1" gate="G$1" pin="(SDA/INT1)PD1"/>
-<wire x1="73.66" y1="2.54" x2="76.2" y2="2.54" width="0.1524" layer="91"/>
-<label x="76.2" y="2.54" size="1.778" layer="95" xref="yes"/>
 </segment>
 </net>
@@
 <junction x="7.62" y="68.58"/>
 <pinref part="X1" gate="G$1" pin="VBUS"/>
-<wire x1="-12.7" y1="12.7" x2="2.54" y2="12.7" width="0.1524" layer="91"/>
-<wire x1="2.54" y1="12.7" x2="2.54" y2="2.54" width="0.1524" layer="91"/>
+<wire x1="-17.78" y1="12.7" x2="-2.54" y2="12.7" width="0.1524" layer="91"/>
+<wire x1="-2.54" y1="12.7" x2="-2.54" y2="2.54" width="0.1524" layer="91"/>
 <pinref part="U$1" gate="G$1" pin="VBUS"/>
-<wire x1="2.54" y1="2.54" x2="7.62" y2="2.54" width="0.1524" layer="91"/>
+<wire x1="-2.54" y1="2.54" x2="7.62" y2="2.54" width="0.1524" layer="91"/>
 <wire x1="7.62" y1="2.54" x2="12.7" y2="2.54" width="0.1524" layer="91"/>
 <wire x1="7.62" y1="12.7" x2="7.62" y2="2.54" width="0.1524" layer="91"/>
@@
 <wire x1="0" y1="53.34" x2="-2.54" y2="53.34" width="0.1524" layer="91"/>
 <label x="-2.54" y="53.34" size="1.778" layer="95" rot="R180" xref="yes"/>
+<junction x="0" y="53.34"/>
 </segment>
 </net>
@@
 <pinref part="X1" gate="G$1" pin="D-"/>
 <pinref part="R6" gate="G$1" pin="1"/>
-<wire x1="-12.7" y1="10.16" x2="-10.16" y2="10.16" width="0.1524" layer="91"/>
+<wire x1="-17.78" y1="10.16" x2="-15.24" y2="10.16" width="0.1524" layer="91"/>
 </segment>
 </net>
@@
 <pinref part="R5" gate="G$1" pin="1"/>
 <pinref part="X1" gate="G$1" pin="D+"/>
-<wire x1="-10.16" y1="7.62" x2="-12.7" y2="7.62" width="0.1524" layer="91"/>
+<wire x1="-15.24" y1="7.62" x2="-17.78" y2="7.62" width="0.1524" layer="91"/>
 </segment>
 </net>
@@
 <pinref part="R5" gate="G$1" pin="2"/>
 <pinref part="U$1" gate="G$1" pin="D+"/>
-<wire x1="0" y1="7.62" x2="12.7" y2="7.62" width="0.1524" layer="91"/>
+<wire x1="-5.08" y1="7.62" x2="12.7" y2="7.62" width="0.1524" layer="91"/>
 </segment>
 </net>
@@
 <pinref part="U$1" gate="G$1" pin="D-"/>
 <pinref part="R6" gate="G$1" pin="2"/>
-<wire x1="12.7" y1="10.16" x2="0" y2="10.16" width="0.1524" layer="91"/>
+<wire x1="12.7" y1="10.16" x2="-5.08" y2="10.16" width="0.1524" layer="91"/>
 </segment>
 </net>
@@
 </segment>
 </net>
+<net name="A2" class="0">
+<segment>
+<pinref part="U$1" gate="G$1" pin="(ADC5/TMS)PF5"/>
+<wire x1="73.66" y1="-10.16" x2="76.2" y2="-10.16" width="0.1524" layer="91"/>
+<label x="76.2" y="-10.16" size="1.778" layer="95" xref="yes"/>
+</segment>
+<segment>
+<pinref part="JP1" gate="G$1" pin="2"/>
+<wire x1="119.38" y1="-12.7" x2="116.84" y2="-12.7" width="0.1524" layer="91"/>
+<label x="116.84" y="-12.7" size="1.778" layer="95" rot="R180" xref="yes"/>
+</segment>
+</net>
+<net name="A3" class="0">
+<segment>
+<pinref part="U$1" gate="G$1" pin="(ADC4/TCK)PF4"/>
+<wire x1="76.2" y1="-12.7" x2="73.66" y2="-12.7" width="0.1524" layer="91"/>
+<label x="76.2" y="-12.7" size="1.778" layer="95" xref="yes"/>
+</segment>
+<segment>
+<pinref part="JP1" gate="G$1" pin="1"/>
+<wire x1="119.38" y1="-10.16" x2="116.84" y2="-10.16" width="0.1524" layer="91"/>
+<label x="116.84" y="-10.16" size="1.778" layer="95" rot="R180" xref="yes"/>
+</segment>
+</net>
+<net name="N$9" class="0">
+<segment>
+<pinref part="C4" gate="G$1" pin="2"/>
+<wire x1="0" y1="33.02" x2="5.08" y2="33.02" width="0.1524" layer="91"/>
+<wire x1="5.08" y1="33.02" x2="5.08" y2="15.24" width="0.1524" layer="91"/>
+<pinref part="U$1" gate="G$1" pin="UCAP"/>
+<wire x1="5.08" y1="15.24" x2="12.7" y2="15.24" width="0.1524" layer="91"/>
+</segment>
+</net>

Commit message: Update library name
Parts:
- U$1: device blinkiverse:ARDUINO_LEONARDO-REV3B_SMARTPRJ_ATMEGA32U4-XUMU -> blinkinlabs:ARDUINO_LEONARDO-REV3B_SMARTPRJ_ATMEGA32U4-XUMU
Changed lines of the file:
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@@
 <?xml version="1.0" encoding="utf-8"?>
 <!DOCTYPE eagle SYSTEM "eagle.dtd">
-<eagle version="6.2">
+<eagle version="6.5.0">
 <drawing>
 <settings>
@@
 <part name="P+5" library="supply1" deviceset="VCC" device=""/>
 <part name="GND10" library="supply1" deviceset="GND" device=""/>
-<part name="U$1" library="blinkiverse" deviceset="ARDUINO_LEONARDO-REV3B_SMARTPRJ_ATMEGA32U4-XU" device="MU"/>
+<part name="U$1" library="blinkinlabs" deviceset="ARDUINO_LEONARDO-REV3B_SMARTPRJ_ATMEGA32U4-XU" device="MU"/>
 <part name="P+1" library="supply1" deviceset="VCC" device=""/>
 <part name="GND1" library="supply1" deviceset="GND" device=""/>

Commit message: RevB, as submitted
Parts:
- removed J1: RS485, con-amp:520426-4
- removed JP1: (no value), SparkFun:M02PTH
- added J3: (no value), con-amp:555153-1
- added U$3: (no value), blinkinlabs:BUTTON_MOMENTARY
- C1, C2, C4, C5, C6, C7: device SparkFun:CAP0805 -> adafruit:C-USC0603
- C3: value .1uF -> 100nF; device SparkFun:CAP0805 -> adafruit:C-USC0603
- Q1: device blinkyboard:CRYSTAL -> blinkinlabs:CRYSTAL_4PAD2520
- R1, R2, R3, R4, R5, R6, R8: device SparkFun:RESISTOR -> adafruit:R-US_R0603
- U$1: value ARDUINO_LEONARDO-REV3B_SMARTPRJ_ATMEGA32U4-XUMU -> ARDUINO_LEONARDO-REV3B_SMARTPRJ_ATMEGA32U4-XUMU_LONG; device blinkinlabs:ARDUINO_LEONARDO-REV3B_SMARTPRJ_ATMEGA32U4-XUMU -> blinkinlabs:ARDUINO_LEONARDO-REV3B_SMARTPRJ_ATMEGA32U4-XUMU_LONG
Connections:
- removed net A2: JP1.2, U$1.(ADC5/TMS)PF5
- removed net A3: JP1.1, U$1.(ADC4/TCK)PF4
- new net RXLED: U$1.(SS/PCINT0)PB0
- new net TXLED: U$1.(XCK1/#CTS)PD5
- net GND: now also C1.2, C2.2, C3.2, C4.2, C5.2, C6.2, C7.2, J3.7, J3.8, Q1.P$1, U$3.P; no longer C1.1, C2.1, C3.1, C4.1, C5.1, C6.1, C7.1, J1.7, J1.8
- net N$2: now also C1.1; no longer C1.2
- net N$5: now also C2.1; no longer C2.2
- net N$9: now also C4.1; no longer C4.2
- net RESET: now also U$3.S
- net RS485A: now also J3.1; no longer J1.1
- net RS485B: now also J3.2; no longer J1.2
- net VCC: now also C3.1, C5.1, C6.1, C7.1; no longer C3.2, C5.2, C6.2, C7.2
- net VMOT: now also J3.4, J3.5; no longer J1.4, J1.5
Other:
- note removed: "EXTRA"
- moved on the sheet: C1, C2, C3, C4, C5, C6, C7
